Commit message: Compelete serial_driver and camera_core

File: auto_aim/src/sentry/urdf/rm_gimbal.urdf.xacro (robot description, xacro)
@@ -1,5 +1,7 @@
-<?xml version="1.0" encoding="utf-8"?>
+<?xml version="1.0"?>
 <robot name="rm_gimbal"
-  xmlns:xacro="http://ros.org/wiki/xacro">
+       xmlns:xacro="http://ros.org/wiki/xacro">
+<xacro:property name="xyz" value="${xyz}"/>
+<xacro:property name="rpy" value="${rpy}"/>
   <link name="odom" />
   <link name="gimbal_big_link" />
@@ -18,5 +20,5 @@
   <link name="left_camera_link" />
   <joint name="left_camera_joint" type="fixed">
-    <origin xyz="0 0 0.05" rpy="0 0 0" />
+    <origin xyz="${xyz}" rpy="${rpy}" />
     <parent link="gimbal_left_link" />
     <child link="left_camera_link" />
@@ -38,5 +40,5 @@
   <link name="right_camera_link" />
   <joint name="right_camera_joint" type="fixed">
-    <origin xyz="0 0 0.05" rpy="0 0 0" />
+    <origin xyz="${xyz}" rpy="${rpy}" />
     <parent link="gimbal_right_link" />
     <child link="right_camera_link" />

Commit message: compelete serial, camera

File: auto_aim/src/sentry/urdf/rm_gimbal.urdf.xacro (robot description, xacro)
@@ -1,53 +1,61 @@
 <?xml version="1.0"?>
-<robot name="rm_gimbal"
-       xmlns:xacro="http://ros.org/wiki/xacro">
-<xacro:property name="xyz" value="${xyz}"/>
-<xacro:property name="rpy" value="${rpy}"/>
-  <link name="odom" />
-  <link name="gimbal_big_link" />
-  <joint name="gimbal_joint" type="floating">
-    <origin xyz="0 0 0" rpy="0 0 0" />
-    <parent link="odom" />
-    <child link="gimbal_big_link" />
+<robot name="rm_gimbal" xmlns:xacro="http://ros.org/wiki/xacro">
+  <!-- 保留原有属性名 -->
+  <xacro:property name="xyz" default="0 0 0"/>
+  <xacro:property name="rpy" default="0 0 0"/>
+  <!-- 根链接和大云台 -->
+  <link name="odom"/>
+  <link name="gimbal_big_link"/>
+  <joint name="gimbal_joint" type="fixed">
+    <origin xyz="0 0 0" rpy="0 0 0"/>
+    <parent link="odom"/>
+    <child link="gimbal_big_link"/>
   </joint>
-  <link name="gimbal_left_link" />
+  <!-- 左云台：增加固定偏移层 -->
+  <link name="gimbal_left_link_offset"/>
+  <joint name="gimbal_left_offset_joint" type="fixed">
+    <origin xyz="0 0.2 0.1" rpy="0 0 0"/>
+    <parent link="gimbal_big_link"/>
+    <child link="gimbal_left_link_offset"/>
+  </joint>
+  <link name="gimbal_left_link"/>
   <joint name="gimbal_big_to_gimbal_left_joint" type="continuous">
-    <origin xyz="0 0.1 0.05" rpy="0 0 0" />
-    <parent link="gimbal_big_link" />
-    <child link="gimbal_left_link" />
-    <axis xyz="0 0 1" />
+    <origin xyz="0 0 0" rpy="0 0 0"/>
+    <parent link="gimbal_left_link_offset"/>
+    <child link="gimbal_left_link"/>
+    <axis xyz="0 0 1"/>
   </joint>
-  <link name="left_camera_link" />
-  <joint name="left_camera_joint" type="fixed">
-    <origin xyz="${xyz}" rpy="${rpy}" />
-    <parent link="gimbal_left_link" />
-    <child link="left_camera_link" />
-    <axis xyz="0 0 0" />
+  <!-- 右云台：增加固定偏移层 -->
+  <link name="gimbal_right_link_offset"/>
+  <joint name="gimbal_right_offset_joint" type="fixed">
+    <origin xyz="0 -0.2 0.1" rpy="0 0 0"/>
+    <parent link="gimbal_big_link"/>
+    <child link="gimbal_right_link_offset"/>
   </joint>
-  <link name="left_camera_optical_frame" />
-  <joint name="left_camera_optical_joint" type="fixed">
-    <origin xyz="0 0 0" rpy="-1.5708 0 -1.5708" />
-    <parent link="left_camera_link" />
-    <child link="left_camera_optical_frame" />
+  <link name="gimbal_right_link"/>
+  <joint name="gimbal_big_to_gimbal_right_joint" type="continuous">
+    <origin xyz="0 0 0" rpy="0 0 0"/>
+    <parent link="gimbal_right_link_offset"/>
+    <child link="gimbal_right_link"/>
+    <axis xyz="0 0 1"/>
   </joint>
-  <link name="gimbal_right_link" />
-  <joint name="gimbal_big_to_gimbal_right_joint" type="continuous">
-    <origin xyz="0 -0.1 0.05" rpy="0 0 0" />
-    <parent link="gimbal_big_link" />
-    <child link="gimbal_right_link" />
-    <axis xyz="0 0 1" />
-  </joint>
-  <link name="right_camera_link" />
-  <joint name="right_camera_joint" type="fixed">
-    <origin xyz="${xyz}" rpy="${rpy}" />
-    <parent link="gimbal_right_link" />
-    <child link="right_camera_link" />
-    <axis xyz="0 0 0" />
-  </joint>
-  <link name="right_camera_optical_frame" />
-  <joint name="right_camera_optical_joint" type="fixed">
-    <origin xyz="0 0 0" rpy="-1.5708 0 -1.5708" />
-    <parent link="right_camera_link" />
-    <child link="right_camera_optical_frame" />
-  </joint>
+  <!-- 摄像机挂载宏：简化重复 -->
+  <xacro:macro name="camera_chain" params="parent_link camera_link_name camera_joint_name optical_frame_name optical_joint_name">
+    <link name="${camera_link_name}"/>
+    <joint name="${camera_joint_name}" type="fixed">
+      <origin xyz="${xyz}" rpy="${rpy}"/>
+      <parent link="${parent_link}"/>
+      <child link="${camera_link_name}"/>
+      <axis xyz="0 0 0"/>
+    </joint>
+    <link name="${optical_frame_name}"/>
+    <joint name="${optical_joint_name}" type="fixed">
+      <origin xyz="0 0 0" rpy="-1.5708 0 -1.5708"/>
+      <parent link="${camera_link_name}"/>
+      <child link="${optical_frame_name}"/>
+    </joint>
+  </xacro:macro>
+  <!-- 左右摄像机链 -->
+  <xacro:camera_chain parent_link="gimbal_left_link" camera_link_name="left_camera_link" camera_joint_name="left_camera_joint" optical_frame_name="left_camera_optical_frame" optical_joint_name="left_camera_optical_joint"/>
+  <xacro:camera_chain parent_link="gimbal_right_link" camera_link_name="right_camera_link" camera_joint_name="right_camera_joint" optical_frame_name="right_camera_optical_frame" optical_joint_name="right_camera_optical_joint"/>
 </robot>

Commit message: 修复若干已知问题

File: auto_aim/src/sentry/urdf/rm_gimbal.urdf.xacro (robot description, xacro)
@@ -15,5 +15,5 @@
   <link name="gimbal_left_link_offset"/>
   <joint name="gimbal_left_offset_joint" type="fixed">
-    <origin xyz="0 0.2 0.1" rpy="0 0 0"/>
+    <origin xyz="0.4229 0.20951 0.15318" rpy="0 0 0"/>
     <parent link="gimbal_big_link"/>
     <child link="gimbal_left_link_offset"/>
@@ -29,5 +29,5 @@
   <link name="gimbal_right_link_offset"/>
   <joint name="gimbal_right_offset_joint" type="fixed">
-    <origin xyz="0 -0.2 0.1" rpy="0 0 0"/>
+    <origin xyz="0.03382 -0.20951 0.15527" rpy="0 0 0"/>
     <parent link="gimbal_big_link"/>
     <child link="gimbal_right_link_offset"/>
@@ -47,9 +47,8 @@
       <parent link="${parent_link}"/>
       <child link="${camera_link_name}"/>
-      <axis xyz="0 0 0"/>
     </joint>
     <link name="${optical_frame_name}"/>
     <joint name="${optical_joint_name}" type="fixed">
-      <origin xyz="0 0 0" rpy="-1.5708 0 -1.5708"/>
+       <origin xyz="0.04 0 0.02" rpy="-1.5708 0 -1.5708"/>
       <parent link="${camera_link_name}"/>
       <child link="${optical_frame_name}"/>

Commit message: update

File: auto_aim/src/sentry/urdf/rm_gimbal.urdf.xacro (robot description, xacro)
@@ -15,5 +15,5 @@
   <link name="gimbal_left_link_offset"/>
   <joint name="gimbal_left_offset_joint" type="fixed">
-    <origin xyz="0.4229 0.20951 0.15318" rpy="0 0 0"/>
+    <origin xyz="0.04229 0.20951 0.15318" rpy="0 0 0"/>
     <parent link="gimbal_big_link"/>
     <child link="gimbal_left_link_offset"/>

Commit message: update

File: auto_aim/src/sentry/urdf/rm_gimbal.urdf.xacro (robot description, xacro)
@@ -1,7 +1,4 @@
 <?xml version="1.0"?>
-<robot name="rm_gimbal" xmlns:xacro="http://ros.org/wiki/xacro">
-  <!-- 保留原有属性名 -->
-  <xacro:property name="xyz" default="0 0 0"/>
-  <xacro:property name="rpy" default="0 0 0"/>
+<robot name="rm_gimbal">
   <!-- 根链接和大云台 -->
   <link name="odom"/>
@@ -40,21 +37,29 @@
     <axis xyz="0 0 1"/>
   </joint>
-  <!-- 摄像机挂载宏：简化重复 -->
-  <xacro:macro name="camera_chain" params="parent_link camera_link_name camera_joint_name optical_frame_name optical_joint_name">
-    <link name="${camera_link_name}"/>
-    <joint name="${camera_joint_name}" type="fixed">
-      <origin xyz="${xyz}" rpy="${rpy}"/>
-      <parent link="${parent_link}"/>
-      <child link="${camera_link_name}"/>
-    </joint>
-    <link name="${optical_frame_name}"/>
-    <joint name="${optical_joint_name}" type="fixed">
-       <origin xyz="0.04 0 0.02" rpy="-1.5708 0 -1.5708"/>
-      <parent link="${camera_link_name}"/>
-      <child link="${optical_frame_name}"/>
-    </joint>
-  </xacro:macro>
-  <!-- 左右摄像机链 -->
-  <xacro:camera_chain parent_link="gimbal_left_link" camera_link_name="left_camera_link" camera_joint_name="left_camera_joint" optical_frame_name="left_camera_optical_frame" optical_joint_name="left_camera_optical_joint"/>
-  <xacro:camera_chain parent_link="gimbal_right_link" camera_link_name="right_camera_link" camera_joint_name="right_camera_joint" optical_frame_name="right_camera_optical_frame" optical_joint_name="right_camera_optical_joint"/>
+  <!-- 左摄像头链 -->
+  <link name="left_camera_link"/>
+  <joint name="left_camera_joint" type="fixed">
+    <origin xyz="0.09733 0 0.01" rpy="0 0 0"/>
+    <parent link="gimbal_left_link"/>
+    <child link="left_camera_link"/>
+  </joint>
+  <link name="left_camera_optical_frame"/>
+  <joint name="left_camera_optical_joint" type="fixed">
+    <origin xyz="0.0 0 0.0" rpy="-1.5708 0 -1.5708"/>
+    <parent link="left_camera_link"/>
+    <child link="left_camera_optical_frame"/>
+  </joint>
+  <!-- 右摄像头链 -->
+  <link name="right_camera_link"/>
+  <joint name="right_camera_joint" type="fixed">
+    <origin xyz="0.09733 0 0.01" rpy="0 0 0"/>
+    <parent link="gimbal_right_link"/>
+    <child link="right_camera_link"/>
+  </joint>
+  <link name="right_camera_optical_frame"/>
+  <joint name="right_camera_optical_joint" type="fixed">
+    <origin xyz="0.0 0 0.0" rpy="-1.5708 0 -1.5708"/>
+    <parent link="right_camera_link"/>
+    <child link="right_camera_optical_frame"/>
+  </joint>
 </robot>
